File: Project Canary V4.6.sch (EAGLE design)
At the start: 61 parts, among them IC2 ATMEGA324PA

Commit message: Added ground to pin 5, (bottom right)
Connections:
- net GND: now also BME280-HEADER.5
Changed lines of the file:
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@@
 <?xml version="1.0" encoding="utf-8"?>
 <!DOCTYPE eagle SYSTEM "eagle.dtd">
-<eagle version="9.2.1">
+<eagle version="8.4.1">
 <drawing>
 <settings>
@@
 <part name="RESET-SW1" library="adafruit" deviceset="SWITCH_PUSHBUTTON" device="SOFTTOUCHSMD_SJ"/>
 <part name="R12" library="adafruit" deviceset="R-US_" device="M0805" value="330"/>
+<part name="GND28" library="supply1" deviceset="GND" device=""/>
 </parts>
 <sheets>
@@
 <attribute name="NAME" x="11.43" y="-21.8186" size="1.778" layer="95" rot="R180"/>
 <attribute name="VALUE" x="11.43" y="-17.018" size="1.778" layer="96" rot="R180"/>
+</instance>
+<instance part="GND28" gate="1" x="238.76" y="17.78" smashed="yes" rot="R180">
+<attribute name="VALUE" x="241.3" y="20.32" size="1.778" layer="96" rot="R180"/>
 </instance>
 </instances>
@@
 <wire x1="0" y1="-20.32" x2="2.54" y2="-20.32" width="0.1524" layer="91"/>
 </segment>
+<segment>
+<pinref part="BME280-HEADER" gate="G$1" pin="5"/>
+<pinref part="GND28" gate="1" pin="GND"/>
+<wire x1="238.76" y1="12.7" x2="238.76" y2="15.24" width="0.1524" layer="91"/>
+</segment>
 </net>

Commit message: Fixed the Ferrite Bead and smoothed out wires
Connections:
- net 5V: now also U$1.2; no longer C25.1, IC2.AVCC, U$1.1
- net N$9: now also C25.1, IC2.AVCC, U$1.1; no longer U$1.2
Changed lines of the file:
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@@
-</segment>
-<segment>
-<pinref part="IC2" gate="G$1" pin="AVCC"/>
-<label x="81.28" y="53.34" size="1.778" layer="95" rot="R180" xref="yes"/>
-<label x="33.02" y="119.38" size="1.778" layer="95" rot="R180" xref="yes"/>
-<pinref part="C25" gate="G$1" pin="1"/>
-<wire x1="88.9" y1="73.66" x2="88.9" y2="55.88" width="0.1524" layer="91"/>
-<pinref part="U$1" gate="G$1" pin="1"/>
-<wire x1="81.28" y1="71.12" x2="81.28" y2="73.66" width="0.1524" layer="91"/>
-<wire x1="81.28" y1="73.66" x2="88.9" y2="73.66" width="0.1524" layer="91"/>
-<junction x="88.9" y="73.66"/>
 </segment>
 <segment>
@@
 <label x="78.74" y="124.46" size="1.778" layer="95" rot="R180" xref="yes"/>
 </segment>
+<segment>
+<pinref part="U$1" gate="G$1" pin="2"/>
+<wire x1="81.28" y1="55.88" x2="81.28" y2="53.34" width="0.1524" layer="91"/>
+<label x="81.28" y="53.34" size="1.778" layer="95"/>
+</segment>
 </net>
 <net name="N$2" class="0">
@@
 </segment>
 </net>
-<net name="N$9" class="0">
-<segment>
-<pinref part="U$1" gate="G$1" pin="2"/>
-<wire x1="81.28" y1="53.34" x2="81.28" y2="55.88" width="0.1524" layer="91"/>
-</segment>
-</net>
 <net name="N$8" class="0">
 <segment>
@@
 </segment>
 </net>
+<net name="N$9" class="0">
+<segment>
+<pinref part="IC2" gate="G$1" pin="AVCC"/>
+<wire x1="88.9" y1="73.66" x2="81.28" y2="73.66" width="0.1524" layer="91"/>
+<pinref part="U$1" gate="G$1" pin="1"/>
+<wire x1="81.28" y1="73.66" x2="81.28" y2="71.12" width="0.1524" layer="91"/>
+<pinref part="C25" gate="G$1" pin="1"/>
+<wire x1="88.9" y1="55.88" x2="88.9" y2="73.66" width="0.1524" layer="91"/>
+<junction x="88.9" y="73.66"/>
+</segment>
+</net>
